File: hardware/hdmizness/hdmizness.sch (KiCad schematic (older format))
At the start: 65 parts, among them J1 HDMI_A_PCB, J2 USB_A_PCB, SW1 SW_Push, U1 F1C100s, U2 TDA19988, U3 W25Q128JVPIQ, U4 EA3058, Y1 24M

Commit message: hdmizness: Redo HDMI part with SiI9022A
Since I have a stock of 25 of both ICs...
Parts:
- removed U2: TDA19988, Package_DFN_QFN:QFN-64-1EP_9x9mm_P0.5mm_EP4.7x4.7mm, symbol hdmizness:TDA19988
- added C1, C31, C32: 100n, Capacitor_SMD:C_0402_1005Metric, symbol Device:C_Small
- added U2: SiI9022A, hdmizness:QFN-72-1EP_10x10mm_P0.5mm_EP4.7x4.7mm_ThermalVias, symbol hdmizness:SiI9022A
- R11: value 10k -> 4k3
- R15: value 200k -> 100k
Connections:
- net +1V8 is gone; now on net +1V2: C2.2, C24.2, C3.2, C4.2, C5.2, C6.2, C7.2, L2.2, R15.2
- net +1V2: now also U2.12 (CVCC12), U2.26 (CVCC12), U2.42 (CVCC12), U2.47 (CVCC12), U2.5 (CVCC12), U2.53 (CVCC12), U2.60 (AVCC12), U2.66 (AVCC12); no longer C15.1, C17.1, C19.1, C30.2, L4.2, R21.2, U1.22 (VDD-CORE), U1.35 (VDD-CORE), U1.71 (VDD-CORE)
- net +3V3: now also U1.48 (PE1/CSI_VSYNC/LCD_D1/TWI2_SDA/UART0_TX/EINTE1), C1.2, C31.2, C32.2, U2.21 (IOVCC), U2.3 (IOVCC), U2.46 (IOVCC); no longer U1.49 (PE0/CSI_HSYNC/LCD_D0/TWI2_SCK/UART0_RX/EINTE0)
- net CPU_SCL: now also U2.1 (CSCL)
- net CPU_SDA: now also U2.2 (CSDA)
- net GND: now also U1.49 (PE0/CSI_HSYNC/LCD_D0/TWI2_SCK/UART0_RX/EINTE0), C1.1, C31.1, C32.1, U2.11 (D17), U2.13 (D16), U2.20 (D9), U2.23 (D8), U2.31 (D1), U2.32 (D0), U2.43 (CGND), U2.55 (RSVDL), U2.57 (IOGND), U2.63 (AGND), U2.69 (IO_SEL), U2.70 (VDDQ), U2.72 (I2C_A2), U2.EP (GND); no longer U1.48 (PE1/CSI_VSYNC/LCD_D1/TWI2_SDA/UART0_TX/EINTE1)
- net HDMI_CEC: now also U2.71 (CEC_A)
- net HDMI_CK_N: now also U2.58 (TXC_N)
- net HDMI_CK_P: now also U2.59 (TXC_P)
- net HDMI_D0_N: now also U2.61 (TX0_N)
- net HDMI_D0_P: now also U2.62 (TX0_P)
- net HDMI_D1_N: now also U2.64 (TX1_N)
- net HDMI_D1_P: now also U2.65 (TX1_P)
- net HDMI_D2_N: now also U2.67 (TX2_N)
- net HDMI_D2_P: now also U2.68 (TX2_P)
- net HDMI_HPD: now also U2.54 (HPD)
- net HDMI_INT: now also U2.52 (INT)
- net HDMI_SCL: now also U2.49 (DSCL)
- net HDMI_SDA: now also U2.48 (DSDA)
- net I2S_BCLK: now also U2.45 (I2S_SCK)
- net I2S_DO: now also U2.41 (I2S_SD0)
- net I2S_LRCK: now also U2.44 (I2S_WS)
- net RGB_CLK: now also U2.22 (PCLK)
- net RGB_D10: now also U2.19 (D10)
- net RGB_D11: now also U2.18 (D11)
- net RGB_D12: now also U2.17 (D12)
- net RGB_D13: now also U2.16 (D13)
- net RGB_D14: now also U2.15 (D14)
- net RGB_D15: now also U2.14 (D15)
- net RGB_D18: now also U2.10 (D18)
- net RGB_D19: now also U2.9 (D19)
- net RGB_D2: now also U2.30 (D2)
- net RGB_D20: now also U2.8 (D20)
- net RGB_D21: now also U2.7 (D21)
- net RGB_D22: now also U2.6 (D22)
- net RGB_D23: now also U2.4 (D23)
- net RGB_D3: now also U2.29 (D3)
- net RGB_D4: now also U2.28 (D4)
- net RGB_D5: now also U2.27 (D5)
- net RGB_D6: now also U2.25 (D6)
- net RGB_D7: now also U2.24 (D7)
- net RGB_DE: now also U2.33 (DE)
- net RGB_HSYNC: now also U2.34 (HSYNC)
- net RGB_VSYNC: now also U2.35 (VSYNC)
- net at R11.1: now also U2.56 (EXT_SWING)
- net HDMI_~RST: now reaches U1.40 (PE9/CSI_D6/UART2_RTS/SPI1_CLK/EINTE9)
- net HDMI_~RST: now also U2.51 (~RST)
- net HDMI_CDC: now reaches U1.41 (PE8/CSI_D5/UART2_RX/SPI1_MOSI/EINTE8)
- net HDMI_CDC: now also U2.50 (CDC_D)
- new net +1V1: C15.1, C17.1, C19.1, C30.2, L4.2, R21.2, U1.22 (VDD-CORE), U1.35 (VDD-CORE), U1.71 (VDD-CORE)
Other:
- note added: "To simplify BOM, always use a 100k\nresistor for R2.\nVout = 0.6 * (R1 / R2) + 0.6 -> R1 = 100k * (Vout / 0.6 - 1)\n - 3v3: R1 = 450k\n - 2v5: R1 = 333k\n - 1v2: R1 = 100k\n - 1v1: R1 = 83k"
- note removed: "To simplify BOM, always use a 100k\nresistor for R2.\nVout = 0.6 * (R1 / R2) + 0.6 -> R1 = 100k * (Vout / 0.6 - 1)\n - 3v3: R1 = 450k\n - 2v5: R1 = 333k\n - 1v8: R1 = 200k\n - 1v1: R1 = 83k"
- moved on the sheet: C2, C3, C4, C5, C6, C7
