File: hardware/hdmizness-v2/hdmizness.kicad_sch (KiCad schematic)
At the start: 68 parts, among them J1 HDMI_A_PCB, J2 USB_A_PCB, SW1 SW_Push, U1 F1C100s, U2 SiI9022A, U3 W25Q128JVPIQ, U4 EA3058, Y1 24M

Commit message: hardware: don't put soldermask in front of pcb connectors
Parts:
- added TP3: GND, TestPoint:TestPoint_Pad_1.0x1.0mm, symbol Connector:TestPoint_Small
Connections:
- net GND: now also TP3.1
Changed lines of the file:
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@@
 	(wire
 		(pts
+			(xy 82.55 140.97) (xy 82.55 143.51)
+		)
+		(stroke
+			(width 0)
+			(type default)
+		)
+	)
+	(wire
+		(pts
 			(xy 43.18 85.09) (xy 30.48 85.09)
 		)
@@
 					(unit 1)
 				)
+			)
+		)
+	)
+	(symbol
+		(lib_id "Connector:TestPoint_Small")
+		(at 82.55 140.97 0)
+		(mirror x)
+		(unit 1)
+		(exclude_from_sim no)
+		(in_bom yes)
+		(on_board yes)
+		(dnp no)
+		(property "Reference" "TP3"
+			(at 81.3308 139.8016 0)
+			(effects
+				(font
+					(size 1.27 1.27)
+				)
+				(justify right)
+			)
+		)
+		(property "Value" "GND"
+			(at 81.3308 142.113 0)
+			(effects
+				(font
+					(size 1.27 1.27)
+				)
+				(justify right)
+			)
+		)
+		(property "Footprint" "TestPoint:TestPoint_Pad_1.0x1.0mm"
+			(at 87.63 140.97 0)
+			(effects
+				(font
+					(size 1.27 1.27)
+				)
+				(hide yes)
+			)
+		)
+		(property "Datasheet" "~"
+			(at 87.63 140.97 0)
+			(effects
+				(font
+					(size 1.27 1.27)
+				)
+				(hide yes)
+			)
+		)
+		(property "Description" ""
+			(at 82.55 140.97 0)
+			(effects
+				(font
+					(size 1.27 1.27)
+				)
+			)
+		)
+		(pin "1"
+		)
+		(instances
+			(project "hdmizness"
+				(path "/b3363a52-8775-4137-8235-3a8f5d8827fc"
+					(reference "TP3")
+					(unit 1)
+				)
+			)
+		)
+	)
+	(symbol
+		(lib_id "power:GND")
+		(at 82.55 143.51 0)
+		(unit 1)
+		(exclude_from_sim no)
+		(in_bom yes)
+		(on_board yes)
+		(dnp no)
+		(fields_autoplaced yes)
+		(property "Reference" "#PWR055"
+			(at 82.55 149.86 0)
+			(effects
+				(font
+					(size 1.27 1.27)
+				)
+				(hide yes)
+			)
+		)
+		(property "Value" "GND"
+			(at 82.55 147.6431 0)
+			(effects
+				(font
+					(size 1.27 1.27)
+				)
+			)
+		)
+		(property "Footprint" ""
+			(at 82.55 143.51 0)
+			(effects
+				(font
+					(size 1.27 1.27)
+				)
+				(hide yes)
+			)
+		)
+		(property "Datasheet" ""
+			(at 82.55 143.51 0)
+			(effects
+				(font
+					(size 1.27 1.27)
+				)
+				(hide yes)
+			)
+		)
+		(property "Description" "Power symbol creates a global label with name \"GND\" , ground"
+			(at 82.55 143.51 0)
+			(effects
+				(font
+					(size 1.27 1.27)
+				)
+				(hide yes)
+			)
+		)
+		(pin "1"
+		)
+		(instances
+			(project ""
+				(path "/b3363a52-8775-4137-8235-3a8f5d8827fc"
+					(reference "#PWR055")
+					(unit 1)
+				)

Commit message: hardware: update bom with chips now on LCSC
F1C100s, SiI9022A and TDA19988 are now available on LCSC. Set the proper
fields to show them on the BoM.
Parts:
- D1: LCSC P/N (none) -> C158099; MFR P/N (none) -> FC-B1010RGBT-HG
- R15: LCSC P/N C305297 -> C258090; MFR P/N WR04X2003FTL -> RC-02W1003FT
- U1: LCSC P/N (none) -> C1511928; MFR P/N (none) -> F1C100s
- U2: LCSC P/N (none) -> C369565; MFR P/N (none) -> SiI9022A
Changed lines of the file:
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@@
 			)
 		)
+		(property "LCSC P/N" "C1511928"
+			(at 105.41 67.31 0)
+			(effects
+				(font
+					(size 1.27 1.27)
+				)
+				(hide yes)
+			)
+		)
+		(property "MFR P/N" "F1C100s"
+			(at 105.41 67.31 0)
+			(effects
+				(font
+					(size 1.27 1.27)
+				)
+				(hide yes)
+			)
+		)
 		(pin "66"
 		)
@@
 			)
 		)
+		(property "LCSC P/N" "C1511928"
+			(at 271.78 203.2 0)
+			(effects
+				(font
+					(size 1.27 1.27)
+				)
+				(hide yes)
+			)
+		)
+		(property "MFR P/N" "F1C100s"
+			(at 271.78 203.2 0)
+			(effects
+				(font
+					(size 1.27 1.27)
+				)
+				(hide yes)
+			)
+		)
 		(pin "43"
 		)
@@
 			)
 		)
-		(property "LCSC P/N" "C305297"
+		(property "LCSC P/N" "C258090"
 			(at 100.33 220.98 0)
 			(effects
@@
 			)
 		)
-		(property "MFR P/N" "WR04X2003FTL"
+		(property "MFR P/N" "RC-02W1003FT"
 			(at 100.33 220.98 0)
 			(effects
@@
 			)
 		)
+		(property "LCSC P/N" "C158099"
+			(at 40.64 123.19 0)
+			(effects
+				(font
+					(size 1.27 1.27)
+				)
+				(hide yes)
+			)
+		)
+		(property "MFR P/N" "FC-B1010RGBT-HG"
+			(at 40.64 123.19 0)
+			(effects
+				(font
+					(size 1.27 1.27)
+				)
+				(hide yes)
+			)
+		)
 		(pin "2"
 		)
@@
 			)
 		)
+		(property "LCSC P/N" "C369565"
+			(at 257.81 67.31 0)
+			(effects
+				(font
+					(size 1.27 1.27)
+				)
+				(hide yes)
+			)
+		)
+		(property "MFR P/N" "SiI9022A"
+			(at 257.81 67.31 0)
+			(effects
+				(font
+					(size 1.27 1.27)
+				)
+				(hide yes)
+			)
+		)
